File: USB-C_UP1.kicad_sch (KiCad schematic)
At the start: 24 parts, among them J11 USB_C_Receptacle, J12 I2C_HD3SS3220, U22 HD3SS3220IRNHR, U23 TPD4E02B04DQA, U24 TPD4E02B04DQA, U25 TPD4E02B04DQA

Commit message: labels naming fixes, USB Type E connector added
Parts:
- removed C108: 10uF, symbol Device:C
- removed R66: 33k, symbol Device:R
- removed R67: 50k, symbol Device:R
Other:
- note removed: "VBUS Detection"

Commit message: TPS25762 EEPROM connector added
Parts:
- renumbered C102 to C103, C103 to C104, C104 to C105, C105 to C106, C106 to C107, C107 to C108, J11 to J12, J12 to J13, R62 to R64, R63 to R65, R64 to R66, R65 to R67
Other:
- title: (none) -> USB Hub

Commit message: deleted duplicated capacitor
Parts:
- C102: renamed from C103; footprint (none) -> Capacitor_THT:C_Radial_D10.0mm_H16.0mm_P5.00mm
- C103: renamed from C104; footprint (none) -> Capacitor_SMD:C_0402_1005Metric
- C104: renamed from C105; footprint (none) -> Capacitor_SMD:C_0402_1005Metric
- C105: renamed from C106; footprint (none) -> Capacitor_SMD:C_0402_1005Metric
- C106: renamed from C107; footprint (none) -> Capacitor_SMD:C_0402_1005Metric
- C107: renamed from C108; footprint (none) -> Capacitor_SMD:C_0402_1005Metric
- J12: footprint (none) -> Connector_USB:USB_C_Receptacle_Amphenol_12401610E4-2A
- J13: footprint (none) -> Connector_PinHeader_1.27mm:PinHeader_1x03_P1.27mm_Vertical
- JP5: footprint (none) -> Jumper:SolderJumper-2_P1.3mm_Open_RoundedPad1.0x1.5mm
- R64, R65, R66, R67: footprint (none) -> Resistor_SMD:R_0603_1608Metric
- TP10, TP11, TP12, TP13: footprint (none) -> TestPoint:TestPoint_2Pads_Pitch5.08mm_Drill1.3mm
- U22: footprint RNH0030A -> footprints:RNH0030A
Changed lines of the file:
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@@
 			)
 		)
-		(property "Footprint" ""
+		(property "Footprint" "TestPoint:TestPoint_2Pads_Pitch5.08mm_Drill1.3mm"
 			(at 53.34 172.72 0)
 			(effects
@@
 			)
 		)
-		(property "Footprint" "RNH0030A"
+		(property "Footprint" "footprints:RNH0030A"
 			(at 96.52 66.04 0)
 			(effects
@@
 			)
 		)
-		(property "Footprint" ""
+		(property "Footprint" "TestPoint:TestPoint_2Pads_Pitch5.08mm_Drill1.3mm"
 			(at 62.23 175.26 0)
 			(effects
@@
 		(on_board yes)
 		(dnp no)
-		(property "Reference" "C107"
+		(property "Reference" "C106"
 			(at 131.826 72.644 90)
 			(effects
@@
 			)
 		)
-		(property "Footprint" ""
+		(property "Footprint" "Capacitor_SMD:C_0402_1005Metric"
 			(at 134.62 73.66 0)
 			(effects
@@
 			(project "USB_hub"
 				(path "/a2586c28-95f1-49e6-9254-37d7a8473e53/7fe2d266-53fd-4db0-a3a6-d5a75d461820/e4bf2cb2-ae79-4a20-a894-cdf581aefbac"
-					(reference "C107")
+					(reference "C106")
 					(unit 1)
 				)
@@
 			)
 		)
-		(property "Footprint" ""
+		(property "Footprint" "Jumper:SolderJumper-2_P1.3mm_Open_RoundedPad1.0x1.5mm"
 			(at 31.75 187.96 0)
 			(effects
@@
 			)
 		)
-		(property "Footprint" ""
+		(property "Footprint" "TestPoint:TestPoint_2Pads_Pitch5.08mm_Drill1.3mm"
 			(at 24.13 162.56 0)
 			(effects
@@
 		(on_board yes)
 		(dnp no)
-		(property "Reference" "C105"
+		(property "Reference" "C104"
 			(at 131.826 59.944 90)
 			(effects
@@
 			)
 		)
-		(property "Footprint" ""
+		(property "Footprint" "Capacitor_SMD:C_0402_1005Metric"
 			(at 134.62 60.96 0)
 			(effects
@@
 			(project "USB_hub"
 				(path "/a2586c28-95f1-49e6-9254-37d7a8473e53/7fe2d266-53fd-4db0-a3a6-d5a75d461820/e4bf2cb2-ae79-4a20-a894-cdf581aefbac"
-					(reference "C105")
+					(reference "C104")
 					(unit 1)
 				)
@@
 			)
 		)
-		(property "Footprint" ""
+		(property "Footprint" "Resistor_SMD:R_0603_1608Metric"
 			(at 36.068 54.61 90)
 			(effects
@@
 		(on_board yes)
 		(dnp no)
-		(property "Reference" "C106"
+		(property "Reference" "C105"
 			(at 140.716 62.484 90)
 			(effects
@@
 			)
 		)
-		(property "Footprint" ""
+		(property "Footprint" "Capacitor_SMD:C_0402_1005Metric"
 			(at 143.51 63.5 0)
 			(effects
@@
 			(project "USB_hub"
 				(path "/a2586c28-95f1-49e6-9254-37d7a8473e53/7fe2d266-53fd-4db0-a3a6-d5a75d461820/e4bf2cb2-ae79-4a20-a894-cdf581aefbac"
-					(reference "C106")
+					(reference "C105")
 					(unit 1)
 				)
@@
 		(on_board yes)
 		(dnp no)
-		(property "Reference" "C108"
+		(property "Reference" "C107"
 			(at 140.716 75.184 90)
 			(effects
@@
 			)
 		)
-		(property "Footprint" ""
+		(property "Footprint" "Capacitor_SMD:C_0402_1005Metric"
 			(at 143.51 76.2 0)
 			(effects
@@
 			(project "USB_hub"
 				(path "/a2586c28-95f1-49e6-9254-37d7a8473e53/7fe2d266-53fd-4db0-a3a6-d5a75d461820/e4bf2cb2-ae79-4a20-a894-cdf581aefbac"
-					(reference "C108")
+					(reference "C107")
 					(unit 1)
 				)
@@
 			)
 		)
-		(property "Footprint" ""
+		(property "Footprint" "TestPoint:TestPoint_2Pads_Pitch5.08mm_Drill1.3mm"
 			(at 24.13 154.94 0)
 			(effects
@@
 			)
 		)
-		(property "Footprint" ""
+		(property "Footprint" "Resistor_SMD:R_0603_1608Metric"
 			(at 43.688 52.07 90)
 			(effects
@@
 		(dnp no)
 		(fields_autoplaced yes)
-		(property "Reference" "C104"
+		(property "Reference" "C103"
 			(at 36.83 29.2099 0)
 			(effects
@@
 			)
 		)
-		(property "Footprint" ""
+		(property "Footprint" "Capacitor_SMD:C_0402_1005Metric"
 			(at 33.9852 34.29 0)
 			(effects
@@
 			(project "USB_hub"
 				(path "/a2586c28-95f1-49e6-9254-37d7a8473e53/7fe2d266-53fd-4db0-a3a6-d5a75d461820/e4bf2cb2-ae79-4a20-a894-cdf581aefbac"
-					(reference "C104")
+					(reference "C103")
 					(unit 1)
 				)
@@
 			)
 		)
-		(property "Footprint" ""
+		(property "Footprint" "Connector_PinHeader_1.27mm:PinHeader_1x03_P1.27mm_Vertical"
 			(at 21.59 175.26 0)
 			(effects
@@
 			)
 		)
-		(property "Footprint" ""
+		(property "Footprint" "Resistor_SMD:R_0603_1608Metric"
 			(at 50.038 45.72 90)
 			(effects
@@
 			)
 		)
-		(property "Footprint" ""
+		(property "Footprint" "Resistor_SMD:R_0603_1608Metric"
 			(at 49.53 67.818 90)
 			(effects
@@
 			)
 		)
-		(property "Footprint" ""
+		(property "Footprint" "Connector_USB:USB_C_Receptacle_Amphenol_12401610E4-2A"
 			(at 245.11 50.8 0)
 			(effects
@@
 		(dnp no)
 		(fields_autoplaced yes)
-		(property "Reference" "C103"
+		(property "Reference" "C102"
 			(at 24.13 29.2099 0)
 			(effects
@@
 			)
 		)
-		(property "Footprint" ""
+		(property "Footprint" "Capacitor_THT:C_Radial_D10.0mm_H16.0mm_P5.00mm"
 			(at 21.2852 34.29 0)
 			(effects
@@
 			(project "USB_hub"
 				(path "/a2586c28-95f1-49e6-9254-37d7a8473e53/7fe2d266-53fd-4db0-a3a6-d5a75d461820/e4bf2cb2-ae79-4a20-a894-cdf581aefbac"
-					(reference "C103")
-					(unit 1)
-				)
+					(reference "C102")
+					(unit 1)
+				)

Commit message: Minor fixes
Fixed unclear labelling of buses
Parts:
- R64, R65, R66, R67: footprint Resistor_SMD:R_0603_1608Metric -> Resistor_SMD:R_0402_1005Metric
Changed lines of the file:
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@@
 			)
 		)
-		(property "Footprint" "Resistor_SMD:R_0603_1608Metric"
+		(property "Footprint" "Resistor_SMD:R_0402_1005Metric"
 			(at 36.068 54.61 90)
 			(effects
@@
 			)
 		)
-		(property "Footprint" "Resistor_SMD:R_0603_1608Metric"
+		(property "Footprint" "Resistor_SMD:R_0402_1005Metric"
 			(at 43.688 52.07 90)
 			(effects
@@
 			)
 		)
-		(property "Footprint" "Resistor_SMD:R_0603_1608Metric"
+		(property "Footprint" "Resistor_SMD:R_0402_1005Metric"
 			(at 50.038 45.72 90)
 			(effects
@@
 			)
 		)
-		(property "Footprint" "Resistor_SMD:R_0603_1608Metric"
+		(property "Footprint" "Resistor_SMD:R_0402_1005Metric"
 			(at 49.53 67.818 90)
 			(effects

Commit message: Scheme fixes
Fixed wrong connection of SNS pin of U21
USB7206c symbol improved
R7's value fixed
Parts:
- U23, U24, U25: symbol Power_Protection:TPD4E02B04DQA -> Snapeda:TPD4E02B04DQA
Connections:
- net USB-C1.CC1: now also U23.10 (NC)
- net USB-C1.CC2: now also U23.9 (NC)
- net USB-C1.D+: now also U23.6 (NC)
- net USB-C1.D-: now also U23.7 (NC)
- net USB-C1.RX1+: now also U25.9 (NC)
- net USB-C1.RX1-: now also U25.10 (NC)
- net USB-C1.RX2+: now also U24.9 (NC)
- net USB-C1.RX2-: now also U24.10 (NC)
- net USB-C1.TX1+: now also U25.6 (NC)
- net USB-C1.TX1-: now also U25.7 (NC)
- net USB-C1.TX2+: now also U24.6 (NC)
- net USB-C1.TX2-: now also U24.7 (NC)
Changed lines of the file:
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@@
 	)
 	(symbol
-		(lib_id "Power_Protection:TPD4E02B04DQA")
+		(lib_id "Snapeda:TPD4E02B04DQA")
 		(at 262.89 140.97 0)
 		(unit 1)
@@
 	)
 	(symbol
-		(lib_id "Power_Protection:TPD4E02B04DQA")
+		(lib_id "Snapeda:TPD4E02B04DQA")
 		(at 222.25 140.97 0)
 		(unit 1)
@@
 	)
 	(symbol
-		(lib_id "Power_Protection:TPD4E02B04DQA")
+		(lib_id "Snapeda:TPD4E02B04DQA")
 		(at 184.15 139.7 0)
 		(unit 1)

Commit message: MCP19035 changed to MP8795
TPS7A4701xRGW to AP7361C-33E
Led Indicator added
Parts:
- added R87, R88: 4.7k, symbol Device:R
- renumbered U22 to U1, U23 to U22, U24 to U23, U25 to U24
Connections:
- net +3V3: now also R87.1, R88.1
- net I2C_HD3SS3220.SCL: now also R88.2
- net I2C_HD3SS3220.SDA: now also R87.2

Commit message: I2C Addresses added to scheme
Connections:
- net +5V: now also JP5.1 (A)
- net GND: no longer JP5.1 (A)
Other:
- note added: "I2C Address 0x67"
Changed lines of the file:
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@@
 		)
 	)
+	(text "I2C Address 0x67"
+		(exclude_from_sim no)
+		(at 40.64 192.024 0)
+		(effects
+			(font
+				(size 1.27 1.27)
+			)
+		)
+	)
 	(text "ESD Protection"
 		(exclude_from_sim no)
@@
 	(wire
 		(pts
-			(xy 25.4 187.96) (xy 29.21 187.96)
+			(xy 19.05 187.96) (xy 29.21 187.96)
 		)
 		(stroke
@@
 	)
 	(symbol
-		(lib_id "power:GND")
-		(at 25.4 187.96 0)
-		(unit 1)
-		(exclude_from_sim no)
-		(in_bom yes)
-		(on_board yes)
-		(dnp no)
-		(fields_autoplaced yes)
-		(property "Reference" "#PWR0194"
-			(at 25.4 194.31 0)
-			(effects
-				(font
-					(size 1.27 1.27)
-				)
-				(hide yes)
-			)
-		)
-		(property "Value" "GND"
-			(at 25.4 193.04 0)
-			(effects
-				(font
-					(size 1.27 1.27)
-				)
-			)
-		)
-		(property "Footprint" ""
-			(at 25.4 187.96 0)
-			(effects
-				(font
-					(size 1.27 1.27)
-				)
-				(hide yes)
-			)
-		)
-		(property "Datasheet" ""
-			(at 25.4 187.96 0)
-			(effects
-				(font
-					(size 1.27 1.27)
-				)
-				(hide yes)
-			)
-		)
-		(property "Description" "Power symbol creates a global label with name \"GND\" , ground"
-			(at 25.4 187.96 0)
-			(effects
-				(font
-					(size 1.27 1.27)
-				)
-				(hide yes)
-			)
-		)
-		(pin "1"
-		)
-		(instances
-			(project "USB_hub"
-				(path "/a2586c28-95f1-49e6-9254-37d7a8473e53/c482699f-16ee-4a02-bb28-667e2389d2fc"
-					(reference "#PWR0194")
-					(unit 1)
-				)
-			)
-		)
-	)
-	(symbol
 		(lib_id "Device:R")
 		(at 69.85 171.45 0)
@@
 					(unit 1)
 				)
+			)
+		)
+	)
+	(symbol
+		(lib_id "power:+5V")
+		(at 19.05 187.96 0)
+		(unit 1)
+		(exclude_from_sim no)
+		(in_bom yes)
+		(on_board yes)
+		(dnp no)
+		(fields_autoplaced yes)
+		(property "Reference" "#PWR0157"
+			(at 19.05 191.77 0)
+			(effects
+				(font
+					(size 1.27 1.27)
+				)
+				(hide yes)
+			)
+		)
+		(property "Value" "+5V"
+			(at 19.05 182.88 0)
+			(effects
+				(font
+					(size 1.27 1.27)
+				)
+			)
+		)
+		(property "Footprint" ""
+			(at 19.05 187.96 0)
+			(effects
+				(font
+					(size 1.27 1.27)
+				)
+				(hide yes)
+			)
+		)
+		(property "Datasheet" ""
+			(at 19.05 187.96 0)
+			(effects
+				(font
+					(size 1.27 1.27)
+				)
+				(hide yes)
+			)
+		)
+		(property "Description" "Power symbol creates a global label with name \"+5V\""
+			(at 19.05 187.96 0)
+			(effects
+				(font
+					(size 1.27 1.27)
+				)
+				(hide yes)
+			)
+		)
+		(pin "1"
+		)
+		(instances
+			(project "USB_hub"
+				(path "/a2586c28-95f1-49e6-9254-37d7a8473e53/c482699f-16ee-4a02-bb28-667e2389d2fc"
+					(reference "#PWR0157")
+					(unit 1)
+				)

Commit message: Ferrite Breads added for 5V, TVS and ESD diodes added
Connections:
- net +5V renamed +5V_USB_C_SD
