File: USB-E_UP.kicad_sch (KiCad schematic)
At the start: 5 parts, among them J14 USB_C_Internal_Connector, U25 TPD4E02B04DQA, U26 TPD4E02B04DQA

Commit message: Schematic reannotated
Parts:
- renumbered R68 to R98, R69 to R99, U25 to U30, U26 to U31
Changed lines of the file:
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@@
 		(dnp no)
 		(fields_autoplaced yes)
-		(property "Reference" "R68"
+		(property "Reference" "R98"
 			(at 203.2 35.5599 0)
 			(effects
@@
 			(project "USB_hub"
 				(path "/a2586c28-95f1-49e6-9254-37d7a8473e53/df13e2b1-cca0-408c-9316-50e440f0b300"
-					(reference "R68")
+					(reference "R98")
 					(unit 1)
 				)
@@
 		(dnp no)
 		(fields_autoplaced yes)
-		(property "Reference" "#PWR0197"
+		(property "Reference" "#PWR0237"
 			(at 209.55 49.53 0)
 			(effects
@@
 			(project "USB_hub"
 				(path "/a2586c28-95f1-49e6-9254-37d7a8473e53/df13e2b1-cca0-408c-9316-50e440f0b300"
-					(reference "#PWR0197")
+					(reference "#PWR0237")
 					(unit 1)
 				)
@@
 		(dnp no)
 		(fields_autoplaced yes)
-		(property "Reference" "#PWR0200"
+		(property "Reference" "#PWR0240"
 			(at 267.97 100.33 0)
 			(effects
@@
 			(project "USB_hub"
 				(path "/a2586c28-95f1-49e6-9254-37d7a8473e53/df13e2b1-cca0-408c-9316-50e440f0b300"
-					(reference "#PWR0200")
+					(reference "#PWR0240")
 					(unit 1)
 				)
@@
 		(on_board yes)
 		(dnp no)
-		(property "Reference" "U25"
+		(property "Reference" "U30"
 			(at 167.64 12.954 0)
 			(effects
@@
 			(project "USB_hub"
 				(path "/a2586c28-95f1-49e6-9254-37d7a8473e53/df13e2b1-cca0-408c-9316-50e440f0b300"
-					(reference "U25")
+					(reference "U30")
 					(unit 1)
 				)
@@
 		(dnp no)
 		(fields_autoplaced yes)
-		(property "Reference" "#PWR0199"
+		(property "Reference" "#PWR0239"
 			(at 175.26 86.36 0)
 			(effects
@@
 			(project "USB_hub"
 				(path "/a2586c28-95f1-49e6-9254-37d7a8473e53/df13e2b1-cca0-408c-9316-50e440f0b300"
-					(reference "#PWR0199")
+					(reference "#PWR0239")
 					(unit 1)
 				)
@@
 		(dnp no)
 		(fields_autoplaced yes)
-		(property "Reference" "#PWR0198"
+		(property "Reference" "#PWR0238"
 			(at 175.26 52.07 0)
 			(effects
@@
 			(project "USB_hub"
 				(path "/a2586c28-95f1-49e6-9254-37d7a8473e53/df13e2b1-cca0-408c-9316-50e440f0b300"
-					(reference "#PWR0198")
+					(reference "#PWR0238")
 					(unit 1)
 				)
@@
 		(dnp no)
 		(fields_autoplaced yes)
-		(property "Reference" "R69"
+		(property "Reference" "R99"
 			(at 212.09 38.0999 0)
 			(effects
@@
 			(project "USB_hub"
 				(path "/a2586c28-95f1-49e6-9254-37d7a8473e53/df13e2b1-cca0-408c-9316-50e440f0b300"
-					(reference "R69")
+					(reference "R99")
 					(unit 1)
 				)
@@
 		(on_board yes)
 		(dnp no)
-		(property "Reference" "U26"
+		(property "Reference" "U31"
 			(at 167.64 47.244 0)
 			(effects
@@
 			(project "USB_hub"
 				(path "/a2586c28-95f1-49e6-9254-37d7a8473e53/df13e2b1-cca0-408c-9316-50e440f0b300"
-					(reference "U26")
+					(reference "U31")
 					(unit 1)
 				)
@@
 		(dnp no)
 		(fields_autoplaced yes)
-		(property "Reference" "#PWR0196"
+		(property "Reference" "#PWR0236"
 			(at 200.66 46.99 0)
 			(effects
@@
 			(project "USB_hub"
 				(path "/a2586c28-95f1-49e6-9254-37d7a8473e53/df13e2b1-cca0-408c-9316-50e440f0b300"
-					(reference "#PWR0196")
+					(reference "#PWR0236")
 					(unit 1)
 				)
@@
 		(on_board no)
 		(dnp no)
-		(property "Reference" "#PWR0195"
+		(property "Reference" "#PWR0235"
 			(at 247.65 30.48 0)
 			(effects
@@
 			(project "USB_hub"
 				(path "/a2586c28-95f1-49e6-9254-37d7a8473e53/df13e2b1-cca0-408c-9316-50e440f0b300"
-					(reference "#PWR0195")
-					(unit 1)
-				)
+					(reference "#PWR0235")
+					(unit 1)
+				)

Commit message: Added lcsc part number for most of components, fixes for better routing
Parts:
- U30, U31: LCSC Part (none) -> C106794
Changed lines of the file:
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@@
+			)
+		)
+		(property "LCSC Part" "C106794"
+			(at 172.72 30.48 0)
+			(effects
+				(font
+					(size 1.27 1.27)
+				)
+				(hide yes)
 			)
 		)
@@
 			(at 172.72 64.77 0)
 			(effects
+				(font
+					(size 1.27 1.27)
+				)
+				(hide yes)
+			)
+		)
+		(property "LCSC Part" "C106794"
+			(at 172.72 64.77 0)
+			(effects

Commit message: Added lcsc part number for most of resistors
Parts:
- R98, R99: LCSC Part (none) -> C2906948
Changed lines of the file:
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@@
+			)
+		)
+		(property "LCSC Part" "C2906948"
+			(at 200.66 36.83 0)
+			(effects
+				(font
+					(size 1.27 1.27)
+				)
+				(hide yes)
 			)
 		)
@@
 			(at 209.55 39.37 0)
 			(effects
+				(font
+					(size 1.27 1.27)
+				)
+				(hide yes)
+			)
+		)
+		(property "LCSC Part" "C2906948"
+			(at 209.55 39.37 0)
+			(effects
