File: USB-A1.kicad_sch (KiCad schematic)
At the start: 23 parts, among them J10 USB3_A, J9 USB3_A, U18 UCS2114-1-V/G4, U19 TPD4E02B04DQA, U20 TPD4E02B04DQA, U32 TPD4E02B04DQA

Commit message: Rearrange of the component placement, scheme changes for better routing
Parts:
- C84: footprint Capacitor_SMD:C_0402_1005Metric -> Capacitor_SMD:C_0201_0603Metric; LCSC Part C5182432 -> C181043
Changed lines of the file:
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@@
 			)
 		)
-		(property "Footprint" "Capacitor_SMD:C_0402_1005Metric"
+		(property "Footprint" "Capacitor_SMD:C_0201_0603Metric"
 			(at 124.1552 26.67 0)
 			(effects
@@
 			)
 		)
-		(property "LCSC Part" "C5182432"
+		(property "LCSC Part" "C181043 "
 			(at 123.19 22.86 0)
 			(effects
