File: USB7206C.kicad_sch (KiCad schematic)
At the start: 42 parts, among them J1 USB_SPI_(Opt), SW1 RESET_HUB, U1 USB7206C/KDX, U2 MIC803-29D4VM3-TR, Y1 25MHz

Commit message: Rearrange of the component placement, scheme changes for better routing
Parts:
- C1, C11, C12, C127, C128, C129, C13, C130, C14, C15, C16, C17, C18, C2, C3, C4, C5, C6, C7, C8, C9: footprint Capacitor_SMD:C_0402_1005Metric -> Capacitor_SMD:C_0201_0603Metric; LCSC Part C5182432 -> C181043
- J1: footprint Connector_PinHeader_1.27mm:PinHeader_1x06_P1.27mm_Vertical -> Connector_PinHeader_1.00mm:PinHeader_1x03_P1.00mm_Vertical; symbol Connector:Conn_01x06_Pin -> Connector:Conn_01x07_Pin
Connections:
- net GND: now also J1.7 (Pin_7)
- net DN2TX-: now reaches C130.1, U1.17 (USB3DN_TXDM2)
- net DN3TX+: now reaches C127.1, U1.29 (USB3DN_TXDP3)
- net DN3TX-: now reaches C128.1, U1.30 (USB3DN_TXDM3)
- net DN2TX+: now reaches C129.1, U1.16 (USB3DN_TXDP2)
Other:
- moved on the sheet: C127, C128, C129, C130
